File: Pi-I2C-Level-Shifter.kicad_pcb (KiCad board)
At the start: 2 copper layers, 27.9 x 15.2 mm, 18 parts, among them J1 Conn_01x05, J2 Conn_02x06_Odd_Even, J4 Conn_01x05, U1 TXB0102DCT, U2 TCA9534

Commit message: Silk edits
Other:
- board text added: "RevA"
- board text removed: "3.3V"
Changed lines of the file:
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@@
   (general
     (thickness 1.6)
-    (drawings 43)
+    (drawings 44)
     (tracks 303)
     (zones 0)
@@
     (tags "solder jumper open")
     (attr virtual)
-    (fp_text reference JP1 (at -2.174 1.397) (layer B.SilkS)
+    (fp_text reference JP1 (at -1.2596 1.651) (layer B.SilkS)
       (effects (font (size 0.9 0.9) (thickness 0.15)) (justify mirror))
     )
@@
       (solder_mask_margin 0.375) (clearance 0.375))
   )
+  (gr_text RevA (at 188.9506 93.2434) (layer B.SilkS)
+    (effects (font (size 1.1 1.1) (thickness 0.15)) (justify mirror))
+  )
   (gr_text . (at 186.7154 84.201) (layer F.SilkS)
     (effects (font (size 1.5 1.5) (thickness 0.3)))
@@
     (effects (font (size 0.9 0.8) (thickness 0.1)))
   )
-  (gr_text 3.3V (at 185.7248 93.1164) (layer B.SilkS)
+  (gr_text 3v3 (at 184.7088 93.2942) (layer B.SilkS)
     (effects (font (size 1.1 1.1) (thickness 0.15)) (justify mirror))
   )
